File: hardware/boards/logger/logger_01.kicad_pcb (KiCad board)
At the start: 2 copper layers, 74 x 20 mm, 49 parts, among them J1 Micro_SD_Card, P1 CONN_01X02, P2 CONN_01X02, P3 Pressure I2C, P4 RTD, T1 1:1 pulse xfmr, U1 LD3985.., U2 Teensy3.2, U4 MCP6072, U5 MCP6072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

Commit message: minor pcb doc changes
Other:
- board text added: "OSH park: Track width 6mil Track spacing 6mil Drilled hole: 10mil min. 5 mil annular ring Min width of solder mask: 4mil circuit to edge: 15mil trace to edge. fine. TODO: SD card too close to edge. Also, no need for slim height part any more."
- board text removed: "OSH park: Track width 6mil Track spacing 6mil Drilled hole: 10mil min. 5 mil annular ring Min width of solder mask: 4mil circuit to edge: 15mil trace to edge. fine."
Changed lines of the file:
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@@
     (links 118)
     (no_connects 0)
-    (area 133.259899 58.22 237.771429 109.81943)
+    (area 133.259899 55.67 282.342857 109.81943)
     (thickness 1.6)
     (drawings 35)
@@
   (page USLetter)
   (layers
-    (0 F.Cu signal hide)
+    (0 F.Cu signal)
     (31 B.Cu signal hide)
     (32 B.Adhes user hide)
@@
     (effects (font (size 1.5 1.5) (thickness 0.3)) (justify mirror))
   )
-  (gr_text "OSH park:\nTrack width 6mil \nTrack spacing 6mil \nDrilled hole: 10mil min.\n5 mil annular ring\nMin width of solder mask: 4mil\n\ncircuit to edge: 15mil trace to edge. fine." (at 188.9 68.3) (layer Cmts.User)
+  (gr_text "OSH park:\nTrack width 6mil \nTrack spacing 6mil \nDrilled hole: 10mil min.\n5 mil annular ring\nMin width of solder mask: 4mil\n\ncircuit to edge: 15mil trace to edge. fine.\n\nTODO: SD card too close to edge.  Also, no need for slim height part any more." (at 188.9 68.3) (layer Cmts.User)
     (effects (font (size 1.5 1.5) (thickness 0.3)) (justify left))
   )
