File: hardware/boards/logger/logger_01.sch (KiCad schematic (older format))
At the start: 50 parts, among them J1 Micro_SD_Card, P1 CONN_01X02, P2 CONN_01X02, P3 CONN_01X04, P4 RTD, T1 1:1 pulse xfmr, U1 LD3985M33R, U2 Teensy3.2, U4 MCP6072, U5 MCP6072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

Commit message: minor pcb doc changes
Other:
- note added: "Add BH123 holder for BOM\nAdd crystal for teensy RTC\nis it safe for en_3v3 not to have a pull-down? might come up floating?"
- note removed: "Add BH123 holder for BOM\nAdd crystal for teensy RTC"
Changed lines of the file:
@@
 LIBS:myparts
 LIBS:teensy
+LIBS:logger_01-cache
 EELAYER 26 0
 EELAYER END
@@
 $EndComp
 Text Notes 700  750  0    60   ~ 0
-Add BH123 holder for BOM\nAdd crystal for teensy RTC
+Add BH123 holder for BOM\nAdd crystal for teensy RTC\nis it safe for en_3v3 not to have a pull-down?  might come up floating?
 $Comp
 L Crystal Y?

Commit message: Long overdue update.
Other:
- note added: "Add BH123 holder for BOM\nAdd crystal for teensy RTC\nis it safe for en_3v3 not to have a pull-down? might come up floating?\nThe AD623s are being used at and beyond their bandwidth! with the\n 10ohm shunt, I tried a 470R gain setting for 200x, which kills the\n performance above 5kHz or so."
- note removed: "Add BH123 holder for BOM\nAdd crystal for teensy RTC\nis it safe for en_3v3 not to have a pull-down? might come up floating?"
Changed lines of the file:
@@
 $EndComp
 Text Notes 700  750  0    60   ~ 0
-Add BH123 holder for BOM\nAdd crystal for teensy RTC\nis it safe for en_3v3 not to have a pull-down?  might come up floating?
+Add BH123 holder for BOM\nAdd crystal for teensy RTC\nis it safe for en_3v3 not to have a pull-down?  might come up floating?\nThe AD623s are being used at and beyond their bandwidth!  with the\n  10ohm shunt, I tried a 470R gain setting for 200x, which kills the\n  performance above 5kHz or so.
 $Comp
 L Crystal Y?
