File: hardware/boards/m0_logger/m0_logger/m0_logger.kicad_pcb (KiCad board)
At the start: 2 copper layers, 94 x 53.3 mm, 17 parts, among them J1 LiPO, J2 PressureA, J3 GPS, J4 PressureB, J5 Micro_SD_Card, U1 MS5803, U2 af_bno055, U3 itsy_m0, U4 DS3231S

Commit message: tweaks
Parts:
- moved J2 1.37 mm to (132.6, 55.4)
- moved J3 1.14 mm to (139.7, 55.4)
Changed lines of the file:
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@@
   )
   (module Connector_PinHeader_2.54mm:PinHeader_2x02_P2.54mm_Horizontal (layer F.Cu)
-    (at 139.7 56.515 270)
+    (at 139.7 55.372 270)
     (descr "Through hole angled pin header, 2x02, 2.54mm pitch, 6mm pin length, double rows")
     (tags "Through hole angled pin header THT 2x02 2.54mm double row")
@@
   )
   (module Connector_PinHeader_2.54mm:PinHeader_2x02_P2.54mm_Horizontal (layer F.Cu)
-    (at 133.35 56.515 270)
+    (at 132.588 55.372 270)
     (descr "Through hole angled pin header, 2x02, 2.54mm pitch, 6mm pin length, double rows")
     (tags "Through hole angled pin header THT 2x02 2.54mm double row")
@@
     (fp_line (start -2.8 -9.85) (end -2.8 9.85) (layer B.Fab) (width 0.15))
     (model "/home/rusty/src/minictd/hardware/parts/Battery Samsung ICR 18650 -22E.step"
-      (offset (xyz -0.5 9.5 17))
+      (offset (xyz -0.5 8.75 17))
       (scale (xyz 1.05 1 1))
       (rotate (xyz 0 0 0))
     )
-  )
+    (model /home/rusty/src/minictd/hardware/housings/pvc-1.25inch.wrl
+      (offset (xyz 0 -0.75 2.3))
+      (scale (xyz 0.394 0.394 0.394))
+      (rotate (xyz 0 -90 0))
+    )
+  )

Commit message: PCB layout sent, minor CAD for housing
Parts:
- added REF**: tab_drills, m0_logger_footprints:tab_drills, F.Cu at (144.8, 63.5)
- added REF**: tab_drills, m0_logger_footprints:tab_drills, F.Cu at (144.8, 69.6)
- moved C1 75.9 mm to (153.0, 62.7)
- moved J4 75.9 mm to (149.9, 61.5)
- moved U1 75.9 mm to (157.5, 62.7)
- moved R2 15.3 mm to (94.1, 57.1), turned to 270 degrees
- moved R1 15.3 mm to (96.6, 57.1), turned to 270 degrees
- moved BT1 15.1 mm to (135.4, 63.2), turned to 270 degrees
- moved J5 2.05 mm to (118.6, 62.0)
- moved J2 1.78 mm to (130.8, 55.4)
- moved U2 1.02 mm to (100.6, 66.0)
- moved J3 0.76 mm to (140.5, 55.4)
- moved C2 0.25 mm to (120.1, 71.9)
- moved C3 0.25 mm to (120.1, 73.9)
Routing:
- net /SD_CS: track 62.0 -> 40.2 mm, vias 4 -> 0
- net Net-(BT1-Pad1): track 38.9 -> 58.9 mm, vias 0 -> 2
- net GND: track 172.1 -> 163.7 mm
- net /MOSI: track 52.8 -> 46.6 mm, vias 4 -> 3
- net /MISO: track 56.5 -> 50.5 mm, vias 4 -> 3
- net /RX: track 62.6 -> 56.7 mm, vias 2 -> 0
- net Net-(J1-Pad1): track 19.8 -> 23.0 mm
- net /SCL: track 79.6 -> 76.7 mm, vias 3 -> 0
- net /SCK: track 57.4 -> 55.3 mm, vias 4 -> 3
- net /TX: track 60.1 -> 58.4 mm, vias 2 -> 0
- net /SDA: track 76.9 -> 75.8 mm, vias 1 -> 2
- net /3V: track 151.3 -> 151.9 mm, vias 3 -> 1
Other:
- board size 94 x 53.3 mm -> 110.5 x 30.5 mm
- net class power added: clearance 0.2, trace_width 0.4, via_dia 0.8, via_drill 0.4
- board text added: "GND +3.6-6V"
- board text added: "Press+IMU+GPS Logger Rusty Holleman 2018-11-28"
- board text added: "slot"
- board text removed: "Bat+ Bat-"

Commit message: Start layout of next board revision
Parts:
- added C5: 0.1uF, Capacitor_SMD:C_0805_2012Metric_Pad1.15x1.40mm_HandSolder, F.Cu at (109.2, 73.9)
- added C6: 2.2uF, Capacitor_SMD:C_0805_2012Metric_Pad1.15x1.40mm_HandSolder, F.Cu at (109.2, 78.2)
- added C7: 47uF, Capacitor_SMD:C_0805_2012Metric_Pad1.15x1.40mm_HandSolder, F.Cu at (106.9, 71.9)
- added C8: 47uF, Capacitor_SMD:C_0805_2012Metric_Pad1.15x1.40mm_HandSolder, F.Cu at (109.2, 75.9)
- added J6: MotA, Connector_Molex:Molex_PicoBlade_53047-0410_1x02_P1.25mm_Vertical, B.Cu at (127.5, 77.5)
- added J7: MotB, Connector_Molex:Molex_PicoBlade_53047-0410_1x02_P1.25mm_Vertical, B.Cu at (121.9, 77.0)
- added J8: Conn_01x03, Connector_PinHeader_2.54mm:PinHeader_1x03_P2.54mm_Vertical, B.Cu at (54.9, 77.2)
- added R3: 0.47, Resistor_SMD:R_0805_2012Metric_Pad1.15x1.40mm_HandSolder, F.Cu at (118.6, 72.1)
- added R4: 0.47, Resistor_SMD:R_0805_2012Metric_Pad1.15x1.40mm_HandSolder, F.Cu at (122.4, 73.4)
- added U5: DRV8833PWP, Package_SO:HTSSOP-16-1EP_4.4x5mm_P0.65mm_EP3.4x5mm_Mask2.46x2.31mm_ThermalVias, F.Cu at (115.6, 76.5)
- J1: moved to B.Cu
- J2, J3: footprint Connector_PinHeader_2.54mm:PinHeader_2x02_P2.54mm_Horizontal -> Connector_Molex:Molex_PicoBlade_53047-0810_1x04_P1.25mm_Vertical; moved to B.Cu
- moved C3 18.2 mm to (112.5, 57.4), turned to 90 degrees
- moved C2 15.6 mm to (114.3, 57.4), turned to 90 degrees
- moved R2 12.8 mm to (81.5, 54.6), turned to 0 degrees
- moved R1 10.9 mm to (86.1, 54.4), turned to 0 degrees
- moved C4 9.07 mm to (112.0, 65.5), turned to 180 degrees
- moved J1 7.88 mm to (63.8, 76.5), turned to 270 degrees
- moved J3 7.87 mm to (140.5, 63.2), turned to 90 degrees
- moved U1 5.30 mm to (159.0, 67.8), turned to 270 degrees
- moved U4 4.75 mm to (97.0, 66.0), turned to 270 degrees
- moved J2 4.34 mm to (132.3, 59.4)
- moved J5 4.13 mm to (122.7, 61.2)
- moved U3 3.94 mm to (70.1, 66.0)
- moved U2 1.27 mm to (101.9, 66.0), turned to 180 degrees
- moved BT1 1.02 mm to (136.4, 63.2)
Connections:
- U3 pad 14: (no net) -> /DRV_nSLEEP
- U3 pad 18: (no net) -> /BIN2
- U3 pad 26: (no net) -> /AIN1
- U3 pad 27: (no net) -> /AIN2
- U3 pad 28: (no net) -> /BIN1
- U3 pad 33: Net-(J1-Pad1) -> /Vbat
Routing:
- net /3V: track 151.9 -> 0.00 mm, vias 1 -> 0
- net GND: track 163.7 -> 30.1 mm, vias 2 -> 0
- net /SCL: track 76.7 -> 0.00 mm
- net /SDA: track 75.8 -> 0.00 mm, vias 2 -> 0
- net Net-(BT1-Pad1): track 58.9 -> 0.00 mm, vias 2 -> 0
- net /TX: track 58.4 -> 0.00 mm
- net /RX: track 56.7 -> 0.00 mm
- net /SCK: track 55.3 -> 0.00 mm, vias 3 -> 0
- net /MISO: track 50.5 -> 0.00 mm, vias 3 -> 0
- net /MOSI: track 46.6 -> 0.00 mm, vias 3 -> 0
- net /SD_CS: track 40.2 -> 0.00 mm
- net Net-(J1-Pad1): track 23.0 -> 0.00 mm
- net /AO1: track 0.00 -> 10.3 mm
- net /DRV_nSLEEP: track 0.00 -> 9.82 mm
- net /AO2: track 0.00 -> 9.25 mm
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Other:
- outline, holes or cut-outs redrawn
- board text added: "DONE add cutout so usb can be plugged even if itsy mounted flush and not on header spacers. DONE drills for itsy and bno055 are too small for standard pins. DONE footprint for ms5803 is somehow shrunk -- way too small. fixed, but double check. DONE Spacing between JST and itsy is tight and makes it difficult to unplug battery. DONE could really use a power switch. 4. GROUND FILL"

Commit message: Finish layout for 2nd revision
Parts:
- moved C2 21.7 mm to (129.8, 72.6)
- moved C3 21.4 mm to (127.5, 72.6)
- moved C4 10.1 mm to (102.9, 61.2), turned to 270 degrees
- moved R2 6.10 mm to (75.4, 54.9)
- moved R1 5.87 mm to (80.3, 54.9)
- moved U4 1.44 mm to (96.0, 65.0)
- moved BT2 1.44 mm to (55.6, 65.8)
Connections:
- U3 pad 18: /BIN2 -> (no net)
- U3 pad 6: (no net) -> /BIN2
Routing:
- net GND: track 30.1 -> 251.6 mm, vias 0 -> 5
- net /3V: track 0.00 -> 177.7 mm, vias 0 -> 1
- net /SCL: track 0.00 -> 102.0 mm, vias 0 -> 3
- net /SDA: track 0.00 -> 91.6 mm, vias 0 -> 3
- net /Vbat: track 7.67 -> 95.5 mm, vias 0 -> 2
- net /TX: track 0.00 -> 64.4 mm, vias 0 -> 2
- net /RX: track 0.00 -> 61.6 mm, vias 0 -> 2
- net /BIN1: track 2.84 -> 63.5 mm, vias 0 -> 3
- net /AIN2: track 4.70 -> 63.4 mm, vias 0 -> 1
- net /BIN2: track 3.68 -> 58.3 mm, vias 0 -> 2
- net /AIN1: track 4.36 -> 58.2 mm, vias 0 -> 1
- net /SCK: track 0.00 -> 50.3 mm, vias 0 -> 2
- net /MISO: track 0.00 -> 47.2 mm, vias 0 -> 2
- net /MOSI: track 0.00 -> 44.2 mm
- net Net-(BT1-Pad1): track 0.00 -> 42.5 mm, vias 0 -> 2
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Other:
- outline, holes or cut-outs redrawn

Commit message: rev2 submitted
Parts:
- removed the C1 at (153.0, 62.7)
- removed the J4 at (149.9, 61.5)
- removed the REF** at (144.8, 63.5)
- removed the REF** at (144.8, 69.6)
- removed the U1 at (159.0, 67.8)
- added C1: 0.1uF, Capacitor_SMD:C_0805_2012Metric_Pad1.15x1.40mm_HandSolder, F.Cu at (153.0, 72.4)
- added C1: 0.1uF, Capacitor_SMD:C_0805_2012Metric_Pad1.15x1.40mm_HandSolder, F.Cu at (153.0, 54.6)
- added J4: PressureB, Connector_PinHeader_2.54mm:PinHeader_1x04_P2.54mm_Vertical, F.Cu at (149.9, 71.1)
- added J4: PressureB, Connector_PinHeader_2.54mm:PinHeader_1x04_P2.54mm_Vertical, F.Cu at (149.9, 53.3)
- added REF**: tab_drills, m0_logger_footprints:tab_drills, F.Cu at (144.8, 73.2)
- added REF**: tab_drills, m0_logger_footprints:tab_drills, F.Cu at (144.8, 79.2)
- added REF**: tab_drills, m0_logger_footprints:tab_drills, F.Cu at (144.8, 55.4)
- added REF**: tab_drills, m0_logger_footprints:tab_drills, F.Cu at (144.8, 61.5)
- added U1: MS5803, m0_logger_footprints:ms5803_rh, B.Cu at (159.0, 77.5)
- added U1: MS5803, m0_logger_footprints:ms5803_rh, B.Cu at (159.0, 59.7)
- moved J7 0.25 mm to (121.7, 77.0)
Connections:
- R3 pad 1: Net-(R3-Pad1) -> /ASEN
- R4 pad 1: Net-(R4-Pad1) -> /BSEN
- U3 pad 8: (no net) -> /ASEN
- U3 pad 9: (no net) -> /BSEN
- U5 pad 3: Net-(R3-Pad1) -> /ASEN
- U5 pad 6: Net-(R4-Pad1) -> /BSEN
Routing:
- net /BSEN: track 0.00 -> 69.8 mm, vias 0 -> 2
- net /ASEN: track 0.00 -> 60.9 mm, vias 0 -> 4
- net /P_GND: track 17.7 -> 35.8 mm, vias 1 -> 2
- net /P_3V: track 16.0 -> 31.9 mm, vias 1 -> 2
- net /P_SCL: track 13.4 -> 26.8 mm, vias 1 -> 2
- net /P_SDA: track 11.4 -> 23.5 mm, vias 1 -> 2
- net Net-(R3-Pad1): track 7.55 -> 0.00 mm, vias 2 -> 0
- net Net-(R4-Pad1): track 4.52 -> 0.00 mm
- net /BIN2: track 58.3 -> 61.6 mm
- net /SCL: track 102.0 -> 100.1 mm
- net /SDA: track 91.6 -> 92.9 mm
- net GND: track 251.6 -> 252.7 mm, vias 5 -> 6
- net /DRV_nSLEEP: track 36.4 -> 35.4 mm
- net /SD_CS: track 40.7 -> 41.6 mm, vias 1 -> 2
- net /MOSI: track 44.2 -> 44.8 mm
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- added copper zone on B.Cu, net GND
Other:
- outline, holes or cut-outs redrawn
- rule via_min_drill: 0.3 -> 0.254
- rule via_min_size: 0.4 -> 0.508
- board text added: "A1,2"
- board text added: "B1,2"
- board text added: "CR1220"
- board text added: "G + SDA SCL"
- board text added: "G V+"
- board text added: "GND + <GPS >GPS"
- board text added: "ON"
- board text added: "Press+IMU+GPS Logger+Mot Rusty Holleman 2018-12-20"
- board text removed: "3V3 >GPS"
- board text removed: "GND +3.6-6V"
- board text removed: "GND <GPS"
- board text removed: "Press+IMU+GPS Logger Rusty Holleman 2018-11-28"
- board text removed: "SCL 3V3"
- board text removed: "SDA GND"
