File: hardware/boards/m0_logger/m0_logger/m0_logger-with_pressure.kicad_pcb (KiCad board)
At the start: 2 copper layers, 94 x 30.5 mm, 24 parts, among them J1 LiPO, J2 PressureA, J3 GPS, J5 Micro_SD_Card, J6 MotA, J7 MotB, J8 Conn_01x03, U2 af_bno055, U3 itsy_m0, U4 DS3231S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

Commit message: Simulation code for buoyancy, config for buoyancy
Parts:
- added C1: 0.1uF, Capacitor_SMD:C_0805_2012Metric_Pad1.15x1.40mm_HandSolder, F.Cu at (153.0, 72.4)
- added C1: 0.1uF, Capacitor_SMD:C_0805_2012Metric_Pad1.15x1.40mm_HandSolder, F.Cu at (153.0, 54.6)
- added J4: PressureB, Connector_PinHeader_2.54mm:PinHeader_1x04_P2.54mm_Vertical, F.Cu at (149.9, 71.1)
- added J4: PressureB, Connector_PinHeader_2.54mm:PinHeader_1x04_P2.54mm_Vertical, F.Cu at (149.9, 53.3)
- added REF**: tab_drills, m0_logger_footprints:tab_drills, F.Cu at (144.8, 73.2)
- added REF**: tab_drills, m0_logger_footprints:tab_drills, F.Cu at (144.8, 79.2)
- added REF**: tab_drills, m0_logger_footprints:tab_drills, F.Cu at (144.8, 55.4)
- added REF**: tab_drills, m0_logger_footprints:tab_drills, F.Cu at (144.8, 61.5)
- added U1: MS5803, m0_logger_footprints:ms5803_rh, B.Cu at (159.0, 77.5)
- added U1: MS5803, m0_logger_footprints:ms5803_rh, B.Cu at (159.0, 59.7)
Routing:
- net /P_GND: track 0.00 -> 35.8 mm, vias 0 -> 2
- net /P_3V: track 0.00 -> 31.9 mm, vias 0 -> 2
- net /P_SCL: track 0.00 -> 26.8 mm, vias 0 -> 2
- net /P_SDA: track 0.00 -> 23.5 mm, vias 0 -> 2
Other:
- board size 94 x 30.5 mm -> 110.5 x 30.5 mm
- board text added: "1. Solder mask on front is missing on the removed pads."
- board text removed: "1. Switch to a beefier JST connector, like the adafruit ones with pads at the front 2. Add a voltage divider to read battery 3. Any way to get the recharging backpack in there? 4. mounting holes if there is room 5. Bevel/chamfer corners to help getting in/out of pipe."
