File: hardware/boards/m0_logger/m0_logger/m0_logger.sch (KiCad schematic (older format))
At the start: 16 parts, among them J1 LiPO, J2 PressureA, J3 GPS, J4 PressureB, J5 Micro_SD_Card, U1 MS5803, U2 af_bno055, U3 itsy_m0, U4 DS3231S

Commit message: Start layout of next board revision
Parts:
- added C5: 0.1uF, Capacitor_SMD:C_0805_2012Metric_Pad1.15x1.40mm_HandSolder, symbol Device:C_Small
- added C6: 2.2uF, Capacitor_SMD:C_0805_2012Metric_Pad1.15x1.40mm_HandSolder, symbol Device:C_Small
- added C7, C8: 47uF, Capacitor_SMD:C_0805_2012Metric_Pad1.15x1.40mm_HandSolder, symbol Device:C_Small
- added J6: MotA, Connector_Molex:Molex_PicoBlade_53047-0410_1x02_P1.25mm_Vertical, symbol Connector_Generic:Conn_01x02
- added J7: MotB, Connector_Molex:Molex_PicoBlade_53047-0410_1x02_P1.25mm_Vertical, symbol Connector_Generic:Conn_01x02
- added J8: Conn_01x03, Connector_PinHeader_2.54mm:PinHeader_1x03_P2.54mm_Vertical, symbol Connector_Generic:Conn_01x03
- added R3, R4: 0.47, Resistor_SMD:R_0805_2012Metric_Pad1.15x1.40mm_HandSolder, symbol Device:R
- added U5: DRV8833PWP, Package_SO:HTSSOP-16-1EP_4.4x5mm_P0.65mm_EP3.4x5mm_Mask2.46x2.31mm_ThermalVias, symbol Driver_Motor:DRV8833PWP
- BT1: Vendor (none) -> 36-500-ND
- C1, C2, C4: Vendor (none) -> 478-1395-1-ND
- C3: Vendor (none) -> 490-9961-1-ND
- J1: Vendor (none) -> 455-1719-ND
- J2, J3: footprint Connector_PinHeader_2.54mm:PinHeader_2x02_P2.54mm_Horizontal -> Connector_Molex:Molex_PicoBlade_53047-0810_1x04_P1.25mm_Vertical; Vendor (none) -> 609-3333-ND
- J4: Vendor (none) -> 609-3255-ND
- J5: Vendor (none) -> HR1964CT-ND
- R1, R2: Vendor (none) -> A126380CT-ND
- U1: Vendor (none) -> 223-1625-5-ND
- U2: Notes (none) -> Also available direct from adafruit; Vendor (none) -> 1528-1426-ND
- U3: Vendor (none) -> 1528-2554-ND
- U4: Vendor (none) -> DS3231S#-ND
Connections:
- net GND: now also C6.2, C7.2, C8.2, R3.2, R4.2, U5.13 (GND), U5.17 (GND(PPAD))
- net DRV_nSLEEP: now reaches U3.14 (D2)
- net DRV_nSLEEP: now also U5.1 (nSLEEP)
- net BIN2: now reaches U3.18 (D3)
- net BIN2: now also U5.10 (BIN2)
- net AIN1: now reaches U3.26 (D9)
- net AIN1: now also U5.16 (AIN1)
- net AIN2: now reaches U3.27 (D10)
- net AIN2: now also U5.15 (AIN2)
- net BIN1: now reaches U3.28 (D11)
- net BIN1: now also U5.9 (BIN1)
- net at J1.1 (Pin_1): now also J8.2 (Pin_2); no longer U3.33 (BAT)
- new net: C5.2, U5.11 (VCP)
- new net: C6.1, U5.14 (VINT)
- new net: R3.1, U5.3 (AISEN)
- new net: R4.1, U5.6 (BISEN)
- new net AO1: J6.1 (Pin_1), U5.2 (AOUT1)
- new net AO2: J6.2 (Pin_2), U5.4 (AOUT2)
- new net BO1: J7.1 (Pin_1), U5.7 (BOUT1)
- new net BO2: J7.2 (Pin_2), U5.5 (BOUT2)
- new net Vbat: C5.1, C7.1, C8.1, J8.1 (Pin_1), U3.33 (BAT), U5.12 (VM)
- no-connect marks 33 -> 30
Other:
- note added: "Mimic Feather\nM0 logger"
- note removed: "Mimic Feather M0 logger"
- moved on the sheet: J1

Commit message: Finish layout for 2nd revision
Connections:
- net BIN2: now also U3.6 (A1); no longer U3.18 (D3)
Changed lines of the file:
@@
 NoConn ~ 5400 2250
 NoConn ~ 5400 2150
-NoConn ~ 5400 2050
 NoConn ~ 5400 1950
 Wire Wire Line
@@
 Wire Wire Line
 	6450 2050 6400 2050
-Text Label 6050 3200 2    50   ~ 0
+Text Label 5200 2050 2    50   ~ 0
 BIN2
-Wire Wire Line
-	6050 3200 6050 3050
 Text Label 4900 2850 0    50   ~ 0
 DRV_nSLEEP
@@
 Text Label 6850 5550 0    50   ~ 0
 BO2
+Wire Wire Line
+	5200 2050 5400 2050
+NoConn ~ 6050 3050
 $EndSCHEMATC

Commit message: rev2 submitted
Connections:
- net ASEN: now reaches U3.8 (A3)
- net ASEN: now also R3.1, U5.3 (AISEN)
- net BSEN: now reaches U3.9 (A4)
- net BSEN: now also R4.1, U5.6 (BISEN)
- no-connect marks 30 -> 28
Changed lines of the file:
@@
 NoConn ~ 6400 1850
 NoConn ~ 5400 2450
-NoConn ~ 5400 2350
-NoConn ~ 5400 2250
 NoConn ~ 5400 2150
 NoConn ~ 5400 1950
@@
 P 5350 4700
 F 0 "C5" H 5250 4800 50  0000 L CNN
-F 1 "0.1uF" H 5200 4600 50  0000 L CNN
+F 1 "0.1uF" H 5350 4600 50  0000 L CNN
 F 2 "Capacitor_SMD:C_0805_2012Metric_Pad1.15x1.40mm_HandSolder" H 5350 4700 50  0001 C CNN
 F 3 "~" H 5350 4700 50  0001 C CNN
@@
 Connection ~ 4850 5050
 Wire Wire Line
-	5250 4950 5600 4950
-Wire Wire Line
-	5600 5050 5250 5050
+	5250 4950 5300 4950
+Wire Wire Line
+	5600 5050 5300 5050
 $Comp
 L Connector_Generic:Conn_01x02 J6
@@
 	5200 2050 5400 2050
 NoConn ~ 6050 3050
+Text Label 5100 2250 0    50   ~ 0
+ASEN
+Text Label 5100 2350 0    50   ~ 0
+BSEN
+Wire Wire Line
+	5100 2250 5400 2250
+Wire Wire Line
+	5400 2350 5100 2350
+Text Label 4650 4750 0    50   ~ 0
+ASEN
+Text Label 4650 5550 0    50   ~ 0
+BSEN
+Wire Wire Line
+	5300 4750 5300 4950
+Connection ~ 5300 4950
+Wire Wire Line
+	5300 4950 5600 4950
+Wire Wire Line
+	5300 5050 5300 5550
+Wire Wire Line
+	5300 5550 4650 5550
+Connection ~ 5300 5050
+Wire Wire Line
+	5300 5050 5250 5050
+Wire Wire Line
+	5300 4750 4650 4750
 $EndSCHEMATC

Commit message: Simulation code for buoyancy, config for buoyancy
Parts:
- C6: Vendor (none) -> 1276-1188-1-ND
- J2, J3: Vendor 609-3333-ND -> WM1733-ND
- J6, J7: Vendor 455-1719-ND -> WM1731-ND
Changed lines of the file:
@@
 F 2 "Connector_Molex:Molex_PicoBlade_53047-0810_1x04_P1.25mm_Vertical" H 1450 5950 50  0001 C CNN
 F 3 "~" H 1450 5950 50  0001 C CNN
-F 4 "609-3333-ND" H 1450 5950 50  0001 C CNN "Vendor"
+F 4 "WM1733-ND" H 1450 5950 50  0001 C CNN "Vendor"
 	1    1450 5950
 	1    0    0    1
@@
 F 2 "Connector_Molex:Molex_PicoBlade_53047-0810_1x04_P1.25mm_Vertical" H 7200 3000 50  0001 C CNN
 F 3 "~" H 7200 3000 50  0001 C CNN
-F 4 "609-3333-ND" H 7200 3000 50  0001 C CNN "Vendor"
+F 4 "WM1733-ND" H 7200 3000 50  0001 C CNN "Vendor"
 	1    7200 3000
 	1    0    0    -1
@@
 F 2 "Capacitor_SMD:C_0805_2012Metric_Pad1.15x1.40mm_HandSolder" H 6900 4400 50  0001 C CNN
 F 3 "~" H 6900 4400 50  0001 C CNN
+F 4 "1276-1188-1-ND" H 6900 4400 50  0001 C CNN "Vendor"
 	1    6900 4400
 	1    0    0    -1
@@
 F 2 "Connector_Molex:Molex_PicoBlade_53047-0410_1x02_P1.25mm_Vertical" H 7350 5250 50  0001 C CNN
 F 3 "~" H 7350 5250 50  0001 C CNN
-F 4 "455-1719-ND" H 7350 5250 50  0001 C CNN "Vendor"
+F 4 "WM1731-ND" H 7350 5250 50  0001 C CNN "Vendor"
 	1    7350 5250
 	1    0    0    -1
@@
 F 2 "Connector_Molex:Molex_PicoBlade_53047-0410_1x02_P1.25mm_Vertical" H 7350 5500 50  0001 C CNN
 F 3 "~" H 7350 5500 50  0001 C CNN
-F 4 "455-1719-ND" H 7350 5500 50  0001 C CNN "Vendor"
+F 4 "WM1731-ND" H 7350 5500 50  0001 C CNN "Vendor"
 	1    7350 5500
 	1    0    0    -1
